File: pcb/matrix.sch (KiCad schematic (older format))
At the start: 88 parts

Commit message: change mcu position, change sw footprint
Parts:
- MX1, MX10, MX11, MX12, MX13, MX14, MX15, MX16, MX17, MX18, MX19, MX2, MX20, MX21, MX22, MX23, MX24, MX25, MX26, MX27, MX28, MX29, MX3, MX30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: footprint MX_Only:MXOnly-1U-Hotswap -> MX_Only:MXOnly-1U-NoLED
- MX41, MX42: footprint MX_Only:MXOnly-1.25U-Hotswap -> MX_Only:MXOnly-1.25U-NoLED
